Commit message: Solving scale error

File: ros2_ws/install/amr_description/share/amr_description/urdf/amr.urdf (robot description, URDF)
Before this commit: robot amr, 5 links, 4 joints
Links:
- removed link l_wheel_link_1
- removed link l_wheel_link_2
- removed link r_wheel_link_1
- removed link r_wheel_link_2
- added link b_wheel_l, mass 0.027390760948486005; collision mesh filename=package://amr_description/meshes/b_wheel_l.stl scale=0.01 0.01 0.01; visual mesh filename=package://amr_description/meshes/b_wheel_l.stl scale=0.01 0.01 0.01
- added link b_wheel_r, mass 0.027390760948486005; collision mesh filename=package://amr_description/meshes/b_wheel_r.stl scale=0.01 0.01 0.01; visual mesh filename=package://amr_description/meshes/b_wheel_r.stl scale=0.01 0.01 0.01
- added link camera_link, mass 0.02186537558266994; collision mesh filename=package://amr_description/meshes/camera_link.stl scale=0.01 0.01 0.01; visual mesh filename=package://amr_description/meshes/camera_link.stl scale=0.01 0.01 0.01
- added link f_wheel_l, mass 0.027390760948486005; collision mesh filename=package://amr_description/meshes/f_wheel_l.stl scale=0.01 0.01 0.01; visual mesh filename=package://amr_description/meshes/f_wheel_l.stl scale=0.01 0.01 0.01
- added link f_wheel_r, mass 0.027390760948486005; collision mesh filename=package://amr_description/meshes/f_wheel_r.stl scale=0.01 0.01 0.01; visual mesh filename=package://amr_description/meshes/f_wheel_r.stl scale=0.01 0.01 0.01
- added link lidar_link, mass 0.030826877913349836; collision mesh filename=package://amr_description/meshes/lidar_link.stl scale=0.01 0.01 0.01; visual mesh filename=package://amr_description/meshes/lidar_link.stl scale=0.01 0.01 0.01
- link base_link: mass 1.202294246159139 -> 1.3304963805212109; geometry collision mesh filename=package://amr_description/meshes/base_link.stl scale=0.01 0.01 0.01; visual mesh filename=package://amr_description/meshes/base_link.stl scale=0.01 0.01 0.01
Joints:
- removed joint base_link_l_wheel_joint_1
- removed joint base_link_l_wheel_joint_2
- removed joint base_link_r_wheel_joint_1
- removed joint base_link_r_wheel_joint_2
- added joint base_link_b_wheel_l_revolute: type continuous, parent base_link, child b_wheel_l, origin xyz=-0.04 0.0425 0.025 rpy=-1.5707963267948966 -0.0 0.0, axis 0.0 0.0 1.0
- added joint base_link_b_wheel_r_revolute: type continuous, parent base_link, child b_wheel_r, origin xyz=-0.04 -0.0425 0.025 rpy=1.5707963267948966 -0.0 0.0, axis 0.0 0.0 1.0
- added joint base_link_camera_rotation: type continuous, parent base_link, child camera_link, origin xyz=0.01916667 0.0 0.055 rpy=0.0 -0.0 0.0, axis 0.0 0.0 1.0
- added joint base_link_f_wheel_l_revolute: type continuous, parent base_link, child f_wheel_l, origin xyz=0.04 0.0425 0.025 rpy=-1.5707963267948966 -0.0 0.0, axis 0.0 0.0 1.0
- added joint base_link_f_wheel_r_revolute: type continuous, parent base_link, child f_wheel_r, origin xyz=0.04 -0.0425 0.025 rpy=1.5707963267948966 -0.0 0.0, axis 0.0 0.0 1.0
- added joint base_link_lidar_rotation: type continuous, parent base_link, child lidar_link, origin xyz=0.0 0.0 0.013000000000000001 rpy=3.141592653589793 -0.0 0.0, axis 0.0 0.0 1.0

File: ros2_ws/install/amr_description/share/amr_description/urdf/amr.xacro (robot description, xacro)
@@ -5,14 +5,15 @@
   <!-- Include gazebo -->
   <xacro:include filename="$(find amr_description)/urdf/gazebo.xacro"/>
+<!--Base Link-->
     <link name="base_link">
         <inertial>
-            <origin xyz="0.0 8.902012997990435e-05 0.0005969174994691003" rpy="0.0 0.0 0.0" />
-            <mass value="1.202294246159139" />
-            <inertia ixx="0.0010272257194446465" iyy="0.0006030855335078637" izz="0.0015348560407595852" ixy="1.070930011337623e-18" iyz="-1.2070886413010125e-06" ixz="0.0" />
+            <origin xyz="-0.0005375575226599613 -6.707584396171594e-18 0.027123229308035738" rpy="0.0 0.0 0.0" />
+            <mass value="1.3304963805212109" />
+            <inertia ixx="0.0006492386077846532" iyy="0.0010792552099575716" izz="0.0015845361638000663" ixy="-7.091559535264415e-19" iyz="-2.420590022530638e-19" ixz="5.575992010655939e-06" />
         </inertial>
         <visual name="base_link_visual">
             <origin xyz="0.0 0.0 0.0" rpy="0.0 0.0 0.0" />
             <geometry>
-                <mesh filename="package://amr_description/meshes/base_link.stl" scale="0.001 0.001 0.001" />
+                <mesh filename="package://amr_description/meshes/base_link.stl" scale="0.01 0.01 0.01" />
             </geometry>
             <material name="base_link"/>
@@ -21,111 +22,165 @@
             <origin xyz="0.0 0.0 0.0" rpy="0.0 0.0 0.0" />
             <geometry>
-                <mesh filename="package://amr_description/meshes/base_link.stl" scale="0.001 0.001 0.001" />
+                <mesh filename="package://amr_description/meshes/base_link.stl" scale="0.01 0.01 0.01" />
             </geometry>
         </collision>
     </link>
-    <link name="r_wheel_link_1">
+<!--Wheels-->
+    <link name="f_wheel_r">
         <inertial>
-            <origin xyz="1.5365486660812167e-14 0.0 -0.04167647058823525" rpy="0.0 -0.0 0.0" />
-            <mass value="0.10481138490538972" />
-            <inertia ixx="1.4602382285722345e-05" iyy="1.4602382288275587e-05" izz="1.9748468661930866e-05" ixy="1.1155520951601516e-20" iyz="-2.710505431213761e-20" ixz="-3.4078799147576644e-17" />
+            <origin xyz="0.0 0.0 0.0075" rpy="0.0 -0.0 0.0" />
+            <mass value="0.027390760948486005" />
+            <inertia ixx="4.793383165985085e-06" iyy="4.793383165984855e-06" izz="8.559612796401754e-06" ixy="0.0" iyz="0.0" ixz="-6.776263578034403e-21" />
         </inertial>
-        <visual name="r_wheel_link_1_visual">
-            <origin xyz="0.0375 -4.440892098500626e-18 0.0" rpy="-1.5707963267948968 -1.5707963267948966 0" />
+        <visual name="f_wheel_r_visual">
+            <origin xyz="-0.04 -0.025 -0.0425" rpy="-1.5707963267948966 -0.0 0.0" />
             <geometry>
-                <mesh filename="package://amr_description/meshes/r_wheel_link_1.stl" scale="0.001 0.001 0.001" />
+                <mesh filename="package://amr_description/meshes/f_wheel_r.stl" scale="0.01 0.01 0.01" />
             </geometry>
             <material name="Wheels"/>
         </visual>
-        <collision name="r_wheel_link_1_collision">
-            <origin xyz="0.0375 -4.440892098500626e-18 0.0" rpy="-1.5707963267948968 -1.5707963267948966 0" />
+        <collision name="f_wheel_r_collision">
+            <origin xyz="-0.04 -0.025 -0.0425" rpy="-1.5707963267948966 -0.0 0.0" />
             <geometry>
-                <mesh filename="package://amr_description/meshes/r_wheel_link_1.stl" scale="0.001 0.001 0.001" />
+                <mesh filename="package://amr_description/meshes/f_wheel_r.stl" scale="0.01 0.01 0.01" />
             </geometry>
         </collision>
     </link>
-    <link name="r_wheel_link_2">
+    <link name="f_wheel_l">
         <inertial>
-            <origin xyz="0.0 -1.537880933710767e-14 -0.04167647058823525" rpy="0.0 -0.0 0.0" />
-            <mass value="0.10481138490538972" />
-            <inertia ixx="1.4602382288275532e-05" iyy="1.4602382285722263e-05" izz="1.9748468661930866e-05" ixy="0.0" iyz="3.412526337898125e-17" ixz="1.1155520951433573e-20" />
+            <origin xyz="0.0 0.0 0.0075" rpy="0.0 -0.0 0.0" />
+            <mass value="0.027390760948486005" />
+            <inertia ixx="4.793383165985099e-06" iyy="4.7933831659848684e-06" izz="8.559612796401754e-06" ixy="0.0" iyz="-6.776263578034403e-21" ixz="-6.776263578034403e-21" />
         </inertial>
-        <visual name="r_wheel_link_2_visual">
-            <origin xyz="-2.220446049250313e-18 0.03749999999999991 3.1086244689504386e-17" rpy="3.141592653589793 -1.570796326794896 0" />
+        <visual name="f_wheel_l_visual">
+            <origin xyz="-0.04 0.025 -0.0425" rpy="1.5707963267948966 -0.0 0.0" />
             <geometry>
-                <mesh filename="package://amr_description/meshes/r_wheel_link_2.stl" scale="0.001 0.001 0.001" />
+                <mesh filename="package://amr_description/meshes/f_wheel_l.stl" scale="0.01 0.01 0.01" />
             </geometry>
             <material name="Wheels"/>
         </visual>
-        <collision name="r_wheel_link_2_collision">
-            <origin xyz="-2.220446049250313e-18 0.03749999999999991 3.1086244689504386e-17" rpy="3.141592653589793 -1.570796326794896 0" />
+        <collision name="f_wheel_l_collision">
+            <origin xyz="-0.04 0.025 -0.0425" rpy="1.5707963267948966 -0.0 0.0" />
             <geometry>
-                <mesh filename="package://amr_description/meshes/r_wheel_link_2.stl" scale="0.001 0.001 0.001" />
+                <mesh filename="package://amr_description/meshes/f_wheel_l.stl" scale="0.01 0.01 0.01" />
             </geometry>
         </collision>
     </link>
-    <link name="l_wheel_link_1">
+    <link name="b_wheel_r">
         <inertial>
-            <origin xyz="0.0 -1.5365486660812167e-14 0.04167647058823525" rpy="0.0 -0.0 0.0" />
-            <mass value="0.10481138490538972" />
-            <inertia ixx="1.4602382288275587e-05" iyy="1.460238228572229e-05" izz="1.974846866193084e-05" ixy="-1.1155520951433573e-20" iyz="-3.4071053270356977e-17" ixz="0.0" />
+            <origin xyz="-8.881784197001253e-18 0.0 0.0075" rpy="0.0 -0.0 0.0" />
+            <mass value="0.027390760948486005" />
+            <inertia ixx="4.793383165985085e-06" iyy="4.793383165984841e-06" izz="8.559612796401754e-06" ixy="-6.776263578034403e-21" iyz="0.0" ixz="-6.776263578034403e-21" />
         </inertial>
-        <visual name="l_wheel_link_1_visual">
-            <origin xyz="4.440892098500626e-18 -0.037500000000000235 -6.217248937900877e-17" rpy="-3.141592653589793 -1.570796326794895 0" />
+        <visual name="b_wheel_r_visual">
+            <origin xyz="0.04 -0.025 -0.0425" rpy="-1.5707963267948966 -0.0 0.0" />
             <geometry>
-                <mesh filename="package://amr_description/meshes/l_wheel_link_1.stl" scale="0.001 0.001 0.001" />
+                <mesh filename="package://amr_description/meshes/b_wheel_r.stl" scale="0.01 0.01 0.01" />
             </geometry>
             <material name="Wheels"/>
         </visual>
-        <collision name="l_wheel_link_1_collision">
-            <origin xyz="4.440892098500626e-18 -0.037500000000000235 -6.217248937900877e-17" rpy="-3.141592653589793 -1.570796326794895 0" />
+        <collision name="b_wheel_r_collision">
+            <origin xyz="0.04 -0.025 -0.0425" rpy="-1.5707963267948966 -0.0 0.0" />
             <geometry>
-                <mesh filename="package://amr_description/meshes/l_wheel_link_1.stl" scale="0.001 0.001 0.001" />
+                <mesh filename="package://amr_description/meshes/b_wheel_r.stl" scale="0.01 0.01 0.01" />
             </geometry>
         </collision>
     </link>
-    <link name="l_wheel_link_2">
+    <link name="b_wheel_l">
         <inertial>
-            <origin xyz="0.0 -1.537880933710767e-14 0.041676470588235245" rpy="0.0 -0.0 0.0" />
-            <mass value="0.10481138490538972" />
-            <inertia ixx="1.4602382288275587e-05" iyy="1.460238228572229e-05" izz="1.9748468661930866e-05" ixy="0.0" iyz="-3.4098158324669114e-17" ixz="0.0" />
+            <origin xyz="-8.881784197001253e-18 0.0 0.0075" rpy="0.0 -0.0 0.0" />
+            <mass value="0.027390760948486005" />
+            <inertia ixx="4.793383165985099e-06" iyy="4.793383165984841e-06" izz="8.559612796401754e-06" ixy="6.776263578034403e-21" iyz="-6.776263578034403e-21" ixz="-1.3552527156068805e-20" />
         </inertial>
-        <visual name="l_wheel_link_2_visual">
-            <origin xyz="0.0 0.03750000000000007 2.6645352591003756e-17" rpy="-3.141592653589793 -1.5707963267948961 0" />
+        <visual name="b_wheel_l_visual">
+            <origin xyz="0.04 0.025 -0.0425" rpy="1.5707963267948966 -0.0 0.0" />
             <geometry>
-                <mesh filename="package://amr_description/meshes/l_wheel_link_2.stl" scale="0.001 0.001 0.001" />
+                <mesh filename="package://amr_description/meshes/b_wheel_l.stl" scale="0.01 0.01 0.01" />
             </geometry>
             <material name="Wheels"/>
         </visual>
-        <collision name="l_wheel_link_2_collision">
-            <origin xyz="0.0 0.03750000000000007 2.6645352591003756e-17" rpy="-3.141592653589793 -1.5707963267948961 0" />
+        <collision name="b_wheel_l_collision">
+            <origin xyz="0.04 0.025 -0.0425" rpy="1.5707963267948966 -0.0 0.0" />
             <geometry>
-                <mesh filename="package://amr_description/meshes/l_wheel_link_2.stl" scale="0.001 0.001 0.001" />
+                <mesh filename="package://amr_description/meshes/b_wheel_l.stl" scale="0.01 0.01 0.01" />
             </geometry>
         </collision>
     </link>
-    <!--Joints-->
-    <joint name="r_wheel_joint_1" type="continuous">
-        <origin xyz="0.0 -0.0375 0.0" rpy="-3.141592653589793 -1.5707963267948966 0" />
+<!--Camera link-->
+    <link name="camera_link">
+        <inertial>
+            <origin xyz="2.1144401675929903e-05 -2.0784716164913716e-18 0.004999999999999991" rpy="0.0 -0.0 0.0" />
+            <mass value="0.02186537558266994" />
+            <inertia ixx="1.6402649642970762e-06" iyy="3.5588437804215866e-07" izz="1.6574154808891354e-06" ixy="2.423405746323952e-19" iyz="-2.0916601783937933e-21" ixz="0.0" />
+        </inertial>
+        <visual name="camera_link_visual">
+            <origin xyz="-0.01916700333333333 1.1102230246251566e-18 -0.055" rpy="0.0 -0.0 0.0" />
+            <geometry>
+                <mesh filename="package://amr_description/meshes/camera_link.stl" scale="0.01 0.01 0.01" />
+            </geometry>
+        </visual>
+        <collision name="camera_link_collision">
+            <origin xyz="-0.01916700333333333 1.1102230246251566e-18 -0.055" rpy="0.0 -0.0 0.0" />
+            <geometry>
+                <mesh filename="package://amr_description/meshes/camera_link.stl" scale="0.01 0.01 0.01" />
+            </geometry>
+            <material name="camera_link"/>
+        </collision>
+    </link>
+<!--Lidar link-->
+    <link name="lidar_link">
+        <inertial>
+            <origin xyz="2.261727773485168e-18 -2.261727773485168e-18 0.003999999999999999" rpy="0.0 -0.0 0.0" />
+            <mass value="0.030826877913349836" />
+            <inertia ixx="1.3685849340280403e-06" iyy="1.3685849340281089e-06" izz="2.4083498369804176e-06" ixy="-2.091660178393795e-21" iyz="4.531930386519889e-22" ixz="-4.531930386519889e-22" />
+        </inertial>
+        <visual name="lidar_link_visual">
+            <origin xyz="0.0 0.0 0.013000000000000001" rpy="3.141592653589793 -0.0 0.0" />
+            <geometry>
+                <mesh filename="package://amr_description/meshes/lidar_link.stl" scale="0.01 0.01 0.01" />
+            </geometry>
+            <material name="lidar_link"/>
+        </visual>
+        <collision name="lidar_link_collision">
+            <origin xyz="0.0 0.0 0.013000000000000001" rpy="3.141592653589793 -0.0 0.0" />
+            <geometry>
+                <mesh filename="package://amr_description/meshes/lidar_link.stl" scale="0.01 0.01 0.01" />
+            </geometry>
+        </collision>
+    </link>
+    <joint name="base_link_f_wheel_r_revolute" type="continuous">
+        <origin xyz="0.04 -0.0425 0.025" rpy="1.5707963267948966 -0.0 0.0" />
         <parent link="base_link" />
-        <child link="r_wheel_link_1" />
+        <child link="f_wheel_r" />
         <axis xyz="0.0 0.0 1.0" />
     </joint>
-    <joint name="l_wheel_joint_1" type="continuous">
-        <origin xyz="0.0 -0.0375 0.0" rpy="-3.141592653589793 -1.5707963267948966 0" />
+    <joint name="base_link_f_wheel_l_revolute" type="continuous">
+        <origin xyz="0.04 0.0425 0.025" rpy="-1.5707963267948966 -0.0 0.0" />
         <parent link="base_link" />
-        <child link="l_wheel_link_1" />
+        <child link="f_wheel_l" />
         <axis xyz="0.0 0.0 1.0" />
     </joint>
-    <joint name="r_wheel_joint_2" type="continuous">
-        <origin xyz="0.0 0.0375 0.0" rpy="-3.141592653589793 -1.5707963267948966 0" />
+    <joint name="base_link_b_wheel_l_revolute" type="continuous">
+        <origin xyz="-0.04 0.0425 0.025" rpy="-1.5707963267948966 -0.0 0.0" />
         <parent link="base_link" />
-        <child link="r_wheel_link_2" />
+        <child link="b_wheel_l" />
         <axis xyz="0.0 0.0 1.0" />
     </joint>
-    <joint name="l_wheel_joint_2" type="continuous">
-        <origin xyz="0.0 0.0375 0.0" rpy="-3.141592653589793 -1.5707963267948966 0" />
+    <joint name="base_link_b_wheel_r_revolute" type="continuous">
+        <origin xyz="-0.04 -0.0425 0.025" rpy="1.5707963267948966 -0.0 0.0" />
         <parent link="base_link" />
-        <child link="l_wheel_link_2" />
+        <child link="b_wheel_r" />
+        <axis xyz="0.0 0.0 1.0" />
+    </joint>
+    <joint name="base_link_camera_rotation" type="continuous">
+        <origin xyz="0.01916667 0.0 0.055" rpy="0.0 -0.0 0.0" />
+        <parent link="base_link" />
+        <child link="camera_link" />
+        <axis xyz="0.0 0.0 1.0" />
+    </joint>
+    <joint name="base_link_lidar_rotation" type="continuous">
+        <origin xyz="0.0 0.0 0.013000000000000001" rpy="3.141592653589793 -0.0 0.0" />
+        <parent link="base_link" />
+        <child link="lidar_link" />
         <axis xyz="0.0 0.0 1.0" />
     </joint>

File: ros2_ws/install/amr_description/share/amr_description/urdf/materials.xacro (robot description, xacro)
@@ -8,3 +8,9 @@
         <color rgba="0.85 0.55 0.1 1"/>
     </material>
+    <material name="camera_link">
+        <color rgba="1 0 0 1"/>
+    </material>
+    <material name="lidar_link">
+        <color rgba="0 1 0 1"/>
+    </material>
 </robot>
