Commit message: The rviz succesfully loaded with amr

File: ros2_ws/install/amr_description/share/amr_description/urdf/amr.urdf (robot description, URDF)
Before this commit: robot amr, 7 links, 6 joints
Links:
- link b_wheel_l: mass 0.027390760948486005 -> 27.390760948486008; geometry collision mesh filename=packages://amr_description/meshes/b_wheel_l.stl scale=0.001 0.001 0.001; visual mesh filename=packages://amr_description/meshes/b_wheel_l.stl scale=0.001 0.001 0.001
- link b_wheel_r: mass 0.027390760948486005 -> 27.390760948486008; geometry collision mesh filename=packages://amr_description/meshes/b_wheel_r.stl scale=0.001 0.001 0.001; visual mesh filename=mpackages://amr_description/eshes/b_wheel_r.stl scale=0.001 0.001 0.001
- link base_link: mass 1.3304963805212109 -> 1330.496380521211; geometry collision mesh filename=packages://amr_description/meshes/base_link.stl scale=0.001 0.001 0.001; visual mesh filename=packages://amr_description/meshes/base_link.stl scale=0.001 0.001 0.001
- link camera_link: mass 0.02186537558266994 -> 21.86537558266994; geometry collision mesh filename=packages://amr_description/meshes/camera_link.stl scale=0.001 0.001 0.001; visual mesh filename=packages://amr_description/meshes/camera_link.stl scale=0.001 0.001 0.001
- link f_wheel_l: mass 0.027390760948486005 -> 27.390760948486008; geometry collision mesh filename=packages://amr_description/meshes/f_wheel_l.stl scale=0.001 0.001 0.001; visual mesh filename=packages://amr_description/meshes/f_wheel_l.stl scale=0.001 0.001 0.001
- link f_wheel_r: mass 0.027390760948486005 -> 27.390760948486008; geometry collision mesh filename=packages://amr_description/meshes/f_wheel_r.stl scale=0.001 0.001 0.001; visual mesh filename=packages://amr_description/meshes/f_wheel_r.stl scale=0.001 0.001 0.001
- link lidar_link: mass 0.030826877913349836 -> 30.826877913349836; geometry collision mesh filename=packages://amr_description/meshes/lidar_link.stl scale=0.001 0.001 0.001; visual mesh filename=packages://amr_description/meshes/lidar_link.stl scale=0.001 0.001 0.001
Joints:
- joint base_link_b_wheel_l_revolute: origin xyz=-0.04 0.0425 0.025 rpy=-1.5707963267948966 -0.0 0.0 -> xyz=-0.4 0.425 -0.065 rpy=-1.5707963267948966 -0.0 0.0
- joint base_link_b_wheel_r_revolute: origin xyz=-0.04 -0.0425 0.025 rpy=1.5707963267948966 -0.0 0.0 -> xyz=-0.4 -0.425 -0.065 rpy=1.5707963267948966 -0.0 0.0
- joint base_link_camera_rotation: origin xyz=0.01916667 0.0 0.055 rpy=0.0 -0.0 0.0 -> xyz=0.19166667 0.0 0.23500000000000001 rpy=0.0 -0.0 0.0
- joint base_link_f_wheel_l_revolute: origin xyz=0.04 0.0425 0.025 rpy=-1.5707963267948966 -0.0 0.0 -> xyz=0.4 0.425 -0.065 rpy=-1.5707963267948966 -0.0 0.0
- joint base_link_f_wheel_r_revolute: origin xyz=0.04 -0.0425 0.025 rpy=1.5707963267948966 -0.0 0.0 -> xyz=0.4 -0.425 -0.065 rpy=1.5707963267948966 -0.0 0.0
- joint base_link_lidar_rotation: origin xyz=0.0 0.0 0.013000000000000001 rpy=3.141592653589793 -0.0 0.0 -> xyz=0.0 0.0 -0.185 rpy=3.141592653589793 -0.0 0.0

File: ros2_ws/install/amr_description/share/amr_description/urdf/amr.xacro (robot description, xacro)
@@ -8,12 +8,12 @@
     <link name="base_link">
         <inertial>
-            <origin xyz="-0.0005375575226599613 -6.707584396171594e-18 0.027123229308035738" rpy="0.0 0.0 0.0" />
-            <mass value="1.3304963805212109" />
-            <inertia ixx="0.0006492386077846532" iyy="0.0010792552099575716" izz="0.0015845361638000663" ixy="-7.091559535264415e-19" iyz="-2.420590022530638e-19" ixz="5.575992010655939e-06" />
+            <origin xyz="-0.005375575226534499 -5.49485313734377e-17 -0.04376770691964268" rpy="0.0 0.0 0.0" />
+            <mass value="1330.496380521211" />
+            <inertia ixx="64.9238607790594" iyy="107.9255209958365" izz="158.45361638099502" ixy="-1.8676558262176537e-13" iyz="-3.189242911227797e-14" ixz="0.5575992010593869" />
         </inertial>
         <visual name="base_link_visual">
             <origin xyz="0.0 0.0 0.0" rpy="0.0 0.0 0.0" />
             <geometry>
-                <mesh filename="package://amr_description/meshes/base_link.stl" scale="0.01 0.01 0.01" />
+                <mesh filename="package://amr_description/meshes/base_link.stl" scale="0.001 0.001 0.001" />
             </geometry>
             <material name="base_link"/>
@@ -22,5 +22,5 @@
             <origin xyz="0.0 0.0 0.0" rpy="0.0 0.0 0.0" />
             <geometry>
-                <mesh filename="package://amr_description/meshes/base_link.stl" scale="0.01 0.01 0.01" />
+                <mesh filename="package://amr_description/meshes/base_link.stl" scale="0.001 0.001 0.001" />
             </geometry>
         </collision>
@@ -29,19 +29,19 @@
     <link name="f_wheel_r">
         <inertial>
-            <origin xyz="0.0 0.0 0.0075" rpy="0.0 -0.0 0.0" />
-            <mass value="0.027390760948486005" />
-            <inertia ixx="4.793383165985085e-06" iyy="4.793383165984855e-06" izz="8.559612796401754e-06" ixy="0.0" iyz="0.0" ixz="-6.776263578034403e-21" />
+            <origin xyz="0.0 3.552713678800501e-17 0.07500000000000007" rpy="0.0 -0.0 0.0" />
+            <mass value="27.390760948486008" />
+            <inertia ixx="0.47933831659850945" iyy="0.4793383165984846" izz="0.8559612796401739" ixy="3.3306690738754696e-16" iyz="-5.551115123125783e-16" ixz="1.7763568394002505e-15" />
         </inertial>
         <visual name="f_wheel_r_visual">
-            <origin xyz="-0.04 -0.025 -0.0425" rpy="-1.5707963267948966 -0.0 0.0" />
-            <geometry>
-                <mesh filename="package://amr_description/meshes/f_wheel_r.stl" scale="0.01 0.01 0.01" />
+            <origin xyz="-0.4 0.065 -0.425" rpy="-1.5707963267948966 -0.0 0.0" />
+            <geometry>
+                <mesh filename="package://amr_description/meshes/f_wheel_r.stl" scale="0.001 0.001 0.001" />
             </geometry>
             <material name="Wheels"/>
         </visual>
         <collision name="f_wheel_r_collision">
-            <origin xyz="-0.04 -0.025 -0.0425" rpy="-1.5707963267948966 -0.0 0.0" />
-            <geometry>
-                <mesh filename="package://amr_description/meshes/f_wheel_r.stl" scale="0.01 0.01 0.01" />
+            <origin xyz="-0.4 0.065 -0.425" rpy="-1.5707963267948966 -0.0 0.0" />
+            <geometry>
+                <mesh filename="package://amr_description/meshes/f_wheel_r.stl" scale="0.001 0.001 0.001" />
             </geometry>
         </collision>
@@ -49,19 +49,19 @@
     <link name="f_wheel_l">
         <inertial>
-            <origin xyz="0.0 0.0 0.0075" rpy="0.0 -0.0 0.0" />
-            <mass value="0.027390760948486005" />
-            <inertia ixx="4.793383165985099e-06" iyy="4.7933831659848684e-06" izz="8.559612796401754e-06" ixy="0.0" iyz="-6.776263578034403e-21" ixz="-6.776263578034403e-21" />
+            <origin xyz="0.0 -3.552713678800501e-17 0.075" rpy="0.0 -0.0 0.0" />
+            <mass value="27.390760948486008" />
+            <inertia ixx="0.4793383165985121" iyy="0.47933831659848636" izz="0.8559612796401739" ixy="-3.3306690738754696e-16" iyz="3.3306690738754696e-16" ixz="0.0" />
         </inertial>
         <visual name="f_wheel_l_visual">
-            <origin xyz="-0.04 0.025 -0.0425" rpy="1.5707963267948966 -0.0 0.0" />
-            <geometry>
-                <mesh filename="package://amr_description/meshes/f_wheel_l.stl" scale="0.01 0.01 0.01" />
+            <origin xyz="-0.4 -0.065 -0.425" rpy="1.5707963267948966 -0.0 0.0" />
+            <geometry>
+                <mesh filename="package://amr_description/meshes/f_wheel_l.stl" scale="0.001 0.001 0.001" />
             </geometry>
             <material name="Wheels"/>
         </visual>
         <collision name="f_wheel_l_collision">
-            <origin xyz="-0.04 0.025 -0.0425" rpy="1.5707963267948966 -0.0 0.0" />
-            <geometry>
-                <mesh filename="package://amr_description/meshes/f_wheel_l.stl" scale="0.01 0.01 0.01" />
+            <origin xyz="-0.4 -0.065 -0.425" rpy="1.5707963267948966 -0.0 0.0" />
+            <geometry>
+                <mesh filename="package://amr_description/meshes/f_wheel_l.stl" scale="0.001 0.001 0.001" />
             </geometry>
         </collision>
@@ -69,19 +69,19 @@
     <link name="b_wheel_r">
         <inertial>
-            <origin xyz="-8.881784197001253e-18 0.0 0.0075" rpy="0.0 -0.0 0.0" />
-            <mass value="0.027390760948486005" />
-            <inertia ixx="4.793383165985085e-06" iyy="4.793383165984841e-06" izz="8.559612796401754e-06" ixy="-6.776263578034403e-21" iyz="0.0" ixz="-6.776263578034403e-21" />
+            <origin xyz="0.0 3.552713678800501e-17 0.07500000000000007" rpy="0.0 -0.0 0.0" />
+            <mass value="27.390760948486008" />
+            <inertia ixx="0.47933831659850945" iyy="0.4793383165984846" izz="0.8559612796401739" ixy="3.3306690738754696e-16" iyz="-5.551115123125783e-16" ixz="-2.6645352591003757e-15" />
         </inertial>
         <visual name="b_wheel_r_visual">
-            <origin xyz="0.04 -0.025 -0.0425" rpy="-1.5707963267948966 -0.0 0.0" />
-            <geometry>
-                <mesh filename="package://amr_description/meshes/b_wheel_r.stl" scale="0.01 0.01 0.01" />
+            <origin xyz="0.4 0.065 -0.425" rpy="-1.5707963267948966 -0.0 0.0" />
+            <geometry>
+                <mesh filename="package://amr_description/meshes/b_wheel_r.stl" scale="0.001 0.001 0.001" />
             </geometry>
             <material name="Wheels"/>
         </visual>
         <collision name="b_wheel_r_collision">
-            <origin xyz="0.04 -0.025 -0.0425" rpy="-1.5707963267948966 -0.0 0.0" />
-            <geometry>
-                <mesh filename="package://amr_description/meshes/b_wheel_r.stl" scale="0.01 0.01 0.01" />
+            <origin xyz="0.4 0.065 -0.425" rpy="-1.5707963267948966 -0.0 0.0" />
+            <geometry>
+                <mesh filename="package://amr_description/meshes/b_wheel_r.stl" scale="0.001 0.001 0.001" />
             </geometry>
         </collision>
@@ -89,19 +89,19 @@
     <link name="b_wheel_l">
         <inertial>
-            <origin xyz="-8.881784197001253e-18 0.0 0.0075" rpy="0.0 -0.0 0.0" />
-            <mass value="0.027390760948486005" />
-            <inertia ixx="4.793383165985099e-06" iyy="4.793383165984841e-06" izz="8.559612796401754e-06" ixy="6.776263578034403e-21" iyz="-6.776263578034403e-21" ixz="-1.3552527156068805e-20" />
+            <origin xyz="0.0 -3.552713678800501e-17 0.075" rpy="0.0 -0.0 0.0" />
+            <mass value="27.390760948486008" />
+            <inertia ixx="0.4793383165985121" iyy="0.47933831659848636" izz="0.8559612796401739" ixy="-3.3306690738754696e-16" iyz="3.3306690738754696e-16" ixz="0.0" />
         </inertial>
         <visual name="b_wheel_l_visual">
-            <origin xyz="0.04 0.025 -0.0425" rpy="1.5707963267948966 -0.0 0.0" />
-            <geometry>
-                <mesh filename="package://amr_description/meshes/b_wheel_l.stl" scale="0.01 0.01 0.01" />
+            <origin xyz="0.4 -0.065 -0.425" rpy="1.5707963267948966 -0.0 0.0" />
+            <geometry>
+                <mesh filename="package://amr_description/meshes/b_wheel_l.stl" scale="0.001 0.001 0.001" />
             </geometry>
             <material name="Wheels"/>
         </visual>
         <collision name="b_wheel_l_collision">
-            <origin xyz="0.04 0.025 -0.0425" rpy="1.5707963267948966 -0.0 0.0" />
-            <geometry>
-                <mesh filename="package://amr_description/meshes/b_wheel_l.stl" scale="0.01 0.01 0.01" />
+            <origin xyz="0.4 -0.065 -0.425" rpy="1.5707963267948966 -0.0 0.0" />
+            <geometry>
+                <mesh filename="package://amr_description/meshes/b_wheel_l.stl" scale="0.001 0.001 0.001" />
             </geometry>
         </collision>
@@ -110,20 +110,20 @@
     <link name="camera_link">
         <inertial>
-            <origin xyz="2.1144401675929903e-05 -2.0784716164913716e-18 0.004999999999999991" rpy="0.0 -0.0 0.0" />
-            <mass value="0.02186537558266994" />
-            <inertia ixx="1.6402649642970762e-06" iyy="3.5588437804215866e-07" izz="1.6574154808891354e-06" ixy="2.423405746323952e-19" iyz="-2.0916601783937933e-21" ixz="0.0" />
+            <origin xyz="0.00021147401675925437 1.1102230246251566e-18 0.05000000000000004" rpy="0.0 -0.0 0.0" />
+            <mass value="21.86537558266994" />
+            <inertia ixx="0.16402649642970402" iyy="0.03558843780421217" izz="0.16574154808891284" ixy="2.4125911295413974e-14" iyz="4.5693013817071915e-17" ixz="2.220446049250313e-16" />
         </inertial>
         <visual name="camera_link_visual">
-            <origin xyz="-0.01916700333333333 1.1102230246251566e-18 -0.055" rpy="0.0 -0.0 0.0" />
-            <geometry>
-                <mesh filename="package://amr_description/meshes/camera_link.stl" scale="0.01 0.01 0.01" />
-            </geometry>
+            <origin xyz="-0.19166700333333336 1.1102230246251566e-18 -0.23500000000000001" rpy="0.0 -0.0 0.0" />
+            <geometry>
+                <mesh filename="package://amr_description/meshes/camera_link.stl" scale="0.001 0.001 0.001" />
+            </geometry>
+            <material name="camera_link"/>
         </visual>
         <collision name="camera_link_collision">
-            <origin xyz="-0.01916700333333333 1.1102230246251566e-18 -0.055" rpy="0.0 -0.0 0.0" />
-            <geometry>
-                <mesh filename="package://amr_description/meshes/camera_link.stl" scale="0.01 0.01 0.01" />
-            </geometry>
-            <material name="camera_link"/>
+            <origin xyz="-0.19166700333333336 1.1102230246251566e-18 -0.23500000000000001" rpy="0.0 -0.0 0.0" />
+            <geometry>
+                <mesh filename="package://amr_description/meshes/camera_link.stl" scale="0.001 0.001 0.001" />
+            </geometry>
         </collision>
     </link>
@@ -131,24 +131,25 @@
     <link name="lidar_link">
         <inertial>
-            <origin xyz="2.261727773485168e-18 -2.261727773485168e-18 0.003999999999999999" rpy="0.0 -0.0 0.0" />
-            <mass value="0.030826877913349836" />
-            <inertia ixx="1.3685849340280403e-06" iyy="1.3685849340281089e-06" izz="2.4083498369804176e-06" ixy="-2.091660178393795e-21" iyz="4.531930386519889e-22" ixz="-4.531930386519889e-22" />
+            <origin xyz="0.0 -1.8528073920390496e-17 0.04" rpy="0.0 -0.0 0.0" />
+            <mass value="30.826877913349836" />
+            <inertia ixx="0.13685849340280387" iyy="0.1368584934028112" izz="0.24083498369804202" ixy="1.8277205526828766e-16" iyz="3.1413946999236946e-17" ixz="0.0" />
         </inertial>
         <visual name="lidar_link_visual">
-            <origin xyz="0.0 0.0 0.013000000000000001" rpy="3.141592653589793 -0.0 0.0" />
-            <geometry>
-                <mesh filename="package://amr_description/meshes/lidar_link.stl" scale="0.01 0.01 0.01" />
+            <origin xyz="0.0 0.0 -0.185" rpy="3.141592653589793 -0.0 0.0" />
+            <geometry>
+                <mesh filename="package://amr_description/meshes/lidar_link.stl" scale="0.001 0.001 0.001" />
             </geometry>
             <material name="lidar_link"/>
         </visual>
         <collision name="lidar_link_collision">
-            <origin xyz="0.0 0.0 0.013000000000000001" rpy="3.141592653589793 -0.0 0.0" />
-            <geometry>
-                <mesh filename="package://amr_description/meshes/lidar_link.stl" scale="0.01 0.01 0.01" />
-            </geometry>
-        </collision>
-    </link>
+            <origin xyz="0.0 0.0 -0.185" rpy="3.141592653589793 -0.0 0.0" />
+            <geometry>
+                <mesh filename="package://amr_description/meshes/lidar_link.stl" scale="0.001 0.001 0.001" />
+            </geometry>
+        </collision>
+    </link>
+<!--Joints-->
     <joint name="base_link_f_wheel_r_revolute" type="continuous">
-        <origin xyz="0.04 -0.0425 0.025" rpy="1.5707963267948966 -0.0 0.0" />
+        <origin xyz="0.4 -0.425 -0.065" rpy="1.5707963267948966 -0.0 0.0" />
         <parent link="base_link" />
         <child link="f_wheel_r" />
@@ -156,5 +157,5 @@
     </joint>
     <joint name="base_link_f_wheel_l_revolute" type="continuous">
-        <origin xyz="0.04 0.0425 0.025" rpy="-1.5707963267948966 -0.0 0.0" />
+        <origin xyz="0.4 0.425 -0.065" rpy="-1.5707963267948966 -0.0 0.0" />
         <parent link="base_link" />
         <child link="f_wheel_l" />
@@ -162,5 +163,5 @@
     </joint>
     <joint name="base_link_b_wheel_l_revolute" type="continuous">
-        <origin xyz="-0.04 0.0425 0.025" rpy="-1.5707963267948966 -0.0 0.0" />
+        <origin xyz="-0.4 0.425 -0.065" rpy="-1.5707963267948966 -0.0 0.0" />
         <parent link="base_link" />
         <child link="b_wheel_l" />
@@ -168,5 +169,5 @@
     </joint>
     <joint name="base_link_b_wheel_r_revolute" type="continuous">
-        <origin xyz="-0.04 -0.0425 0.025" rpy="1.5707963267948966 -0.0 0.0" />
+        <origin xyz="-0.4 -0.425 -0.065" rpy="1.5707963267948966 -0.0 0.0" />
         <parent link="base_link" />
         <child link="b_wheel_r" />
@@ -174,5 +175,5 @@
     </joint>
     <joint name="base_link_camera_rotation" type="continuous">
-        <origin xyz="0.01916667 0.0 0.055" rpy="0.0 -0.0 0.0" />
+        <origin xyz="0.19166667 0.0 0.23500000000000001" rpy="0.0 -0.0 0.0" />
         <parent link="base_link" />
         <child link="camera_link" />
@@ -180,8 +181,60 @@
     </joint>
     <joint name="base_link_lidar_rotation" type="continuous">
-        <origin xyz="0.0 0.0 0.013000000000000001" rpy="3.141592653589793 -0.0 0.0" />
+        <origin xyz="0.0 0.0 -0.185" rpy="3.141592653589793 -0.0 0.0" />
         <parent link="base_link" />
         <child link="lidar_link" />
         <axis xyz="0.0 0.0 1.0" />
     </joint>
+    <!-- Camera Sensor Plugin -->
+        <gazebo reference="camera_link">
+            <sensor name="camera_sensor" type="camera">
+                <update_rate>30.0</update_rate>
+                <camera>
+                    <horizontal_fov>1.047</horizontal_fov>
+                    <image>
+                        <width>640</width>
+                        <height>480</height>
+                        <format>R8G8B8</format>
+                    </image>
+                    <clip>
+                        <near>0.1</near>
+                        <far>100.0</far>
+                    </clip>
+                </camera>
+                <plugin name="camera_controller" filename="libgazebo_ros_camera.so">
+                    <ros>
+                        <namespace>/camera</namespace>
+                    </ros>
+                    <frame_name>camera_link</frame_name>
+                </plugin>
+            </sensor>
+        </gazebo>
+    <!-- LiDAR Sensor Plugin -->
+        <gazebo reference="lidar_link">
+            <sensor name="lidar_sensor" type="ray">
+                <update_rate>10.0</update_rate>
+                <ray>
+                    <scan>
+                        <horizontal>
+                            <samples>720</samples>
+                            <resolution>1</resolution>
+                            <min_angle>-3.14159</min_angle>
+                            <max_angle>3.14159</max_angle>
+                        </horizontal>
+                    </scan>
+                    <range>
+                        <min>0.12</min>
+                        <max>12.0</max>
+                        <resolution>0.01</resolution>
+                    </range>
+                </ray>
+                <plugin name="laser_controller" filename="libgazebo_ros_ray_sensor.so">
+                    <ros>
+                        <remapping>~/out:=scan</remapping>
+                    </ros>
+                    <output_type>sensor_msgs/LaserScan</output_type>
+                    <frame_name>lidar_link</frame_name>
+                </plugin>
+            </sensor>
+        </gazebo>
 </robot>
